File: BatteryCharger/462FinalProject.kicad_pcb (KiCad board)
At the start: 2 copper layers, 30 parts, among them Q1 2N2219, Q2 PMOS, Q3 PMOS, Q4 PMOS, Q5 2N2219, Q6 2N2219, Q7 PMOS, Q8 PMOS, U1 TLV9062xD

Commit message: "Complete" kicad pcb
Parts:
- removed D2, D3, D4: 1N5711, Diode_THT:D_DO-35_SOD27_P7.62mm_Horizontal
- removed H1, H2, H3, H4, H5: MountingHole_Pad, MountingHole:MountingHole_2.1mm
- removed Q5: 2N2219, Package_TO_SOT_THT:TO-39-3
- removed R11: 1k, Resistor_SMD:R_0201_0603Metric
- removed R2, R3, R6, R7: 10k, Resistor_SMD:R_0201_0603Metric
- removed R8: 100m, Resistor_SMD:R_0201_0603Metric
- added C1: 10u, Capacitor_SMD:C_0805_2012Metric_Pad1.18x1.45mm_HandSolder, F.Cu at (206.4, 67.2)
- added C2: 10u, Capacitor_SMD:C_0805_2012Metric_Pad1.18x1.45mm_HandSolder, F.Cu at (206.9, 124.7)
- added C3: 10u, Capacitor_SMD:C_0805_2012Metric_Pad1.18x1.45mm_HandSolder, F.Cu at (206.4, 69.7)
- added C4: .1u, Capacitor_SMD:C_0805_2012Metric_Pad1.18x1.45mm_HandSolder, F.Cu at (206.9, 129.7)
- added C5: 10u, Capacitor_SMD:C_0805_2012Metric_Pad1.18x1.45mm_HandSolder, F.Cu at (206.9, 132.3)
- added C6: 10u, Capacitor_SMD:C_0805_2012Metric_Pad1.18x1.45mm_HandSolder, F.Cu at (206.9, 127.2)
- added D5: MBR0530, Diode_SMD:D_SOD-123, F.Cu at (207.5, 81.6)
- added D6: MBR0530, Diode_SMD:D_SOD-123, F.Cu at (207.5, 84.2)
- added D7: MBR0530, Diode_SMD:D_SOD-123, F.Cu at (207.5, 86.7)
- added IC1: TPS562231DRLR, Library:SOTFL50P160X60-6N, F.Cu at (217.8, 126.6)
- added J2: 3_Pin_Header_to_Battery, Connector_PinHeader_2.54mm:PinHeader_1x03_P2.54mm_Vertical, F.Cu at (228.6, 132.1)
- added J3: USB_B_Micro, Library:USB_Micro-B_roundholes, F.Cu at (230.2, 71.1)
- added J4: 3_Pin_Header_to_IPOD, Connector_PinHeader_2.54mm:PinHeader_1x03_P2.54mm_Vertical, F.Cu at (228.6, 121.9)
- added J5: Conn_01x04_Pin, Connector_PinHeader_2.54mm:PinHeader_1x04_P2.54mm_Vertical, F.Cu at (228.6, 154.9)
- added L2: 3.3u, Library:CC322522A-4R7K, F.Cu at (220.9, 118.1)
- added Q9: SI2302, Package_TO_SOT_SMD:SOT-23, F.Cu at (218.5, 108.1)
- added R12: 1k, Resistor_SMD:R_0805_2012Metric, F.Cu at (206.2, 76.5)
- added RN1: R_Pack04_Split_2, Resistor_SMD:R_Array_Concave_4x0603, F.Cu at (213.6, 97.5)
- added RN2: R_Pack04_Split_2, Resistor_SMD:R_Array_Concave_4x0603, F.Cu at (207.2, 118.2)
- added TP1: TestPoint, TestPoint:TestPoint_Loop_D2.50mm_Drill1.85mm, F.Cu at (204.1, 139.7)
- added TP10: TestPoint, TestPoint:TestPoint_Loop_D2.50mm_Drill1.85mm, F.Cu at (209.5, 139.6)
- added TP2: TestPoint, TestPoint:TestPoint_Loop_D2.50mm_Drill1.85mm, F.Cu at (204.1, 145.1)
- added TP3: TestPoint, TestPoint:TestPoint_Loop_D2.50mm_Drill1.85mm, F.Cu at (204.1, 150.6)
- added TP4: TestPoint, TestPoint:TestPoint_Loop_D2.50mm_Drill1.85mm, F.Cu at (204.1, 156.0)
- added TP5: TestPoint, TestPoint:TestPoint_Loop_D2.50mm_Drill1.85mm, F.Cu at (204.1, 161.5)
- added TP6: TestPoint, TestPoint:TestPoint_Loop_D2.50mm_Drill1.85mm, F.Cu at (209.6, 161.6)
- added TP7: TestPoint, TestPoint:TestPoint_Loop_D2.50mm_Drill1.85mm, F.Cu at (209.5, 145.1)
- added TP8: TestPoint, TestPoint:TestPoint_Loop_D2.50mm_Drill1.85mm, F.Cu at (209.5, 150.6)
- added TP9: TestPoint, TestPoint:TestPoint_Loop_D2.50mm_Drill1.85mm, F.Cu at (209.5, 156.0)
- added U2: STM32G030F6Px, Package_SO:TSSOP-20_4.4x6.5mm_P0.65mm, F.Cu at (219.2, 156.2)
- added U3: ~, Package_SO:SOIC-14_3.9x8.7mm_P1.27mm, F.Cu at (227.2, 143.8)
- D1: value 1N5711 -> MBR0530; footprint Diode_THT:D_DO-35_SOD27_P7.62mm_Horizontal -> Diode_SMD:D_SOD-123
- L1: value 50u -> SRR1205-500YL; footprint Inductor_SMD:L_6.3x6.3_H3 -> Library:SRR1205500YL
- Q1: value 2N2219 -> MMFTN6001; footprint Package_TO_SOT_THT:TO-39-3 -> Package_TO_SOT_SMD:SOT-23
- Q2: value PMOS -> MMFTN6001; footprint Transistor_Power:GaN_Systems_GaNPX-3_5x6.6mm_Drain2.93x0.6mm -> Package_TO_SOT_SMD:SOT-23
- Q3, Q4: value PMOS -> SI2302; footprint Transistor_Power:GaN_Systems_GaNPX-3_5x6.6mm_Drain2.93x0.6mm -> Package_TO_SOT_SMD:SOT-23
- Q6: value 2N2219 -> BSS84AK,215; footprint Package_TO_SOT_THT:TO-39-3 -> Library:SOT95P230X110-3N
- Q7, Q8: value PMOS -> BSS84AK,215; footprint Transistor_Power:GaN_Systems_GaNPX-3_5x6.6mm_Drain2.93x0.6mm -> Library:SOT95P230X110-3N
- R1: value 1k -> 100m; footprint Resistor_SMD:R_0201_0603Metric -> Resistor_SMD:R_0805_2012Metric
- R10: footprint Resistor_SMD:R_0201_0603Metric -> Resistor_SMD:R_0805_2012Metric
- R4: value 10k -> 1k; footprint Resistor_SMD:R_0201_0603Metric -> Resistor_SMD:R_0805_2012Metric
- R5: value 10k -> 45.3k; footprint Resistor_SMD:R_0201_0603Metric -> Library:CR0603-FX-4532ELF
- R9: value 300k -> 100k; footprint Resistor_SMD:R_0201_0603Metric -> Resistor_SMD:R_0805_2012Metric
- U1: value TLV9062xD -> MIC5504-3.3YM5; footprint Package_SO:SOIC-8_3.9x4.9mm_P1.27mm -> Package_TO_SOT_SMD:SOT-23-5
- moved Q2 203.2 mm to (222.6, 108.1), turned to -90 degrees
- moved R1 196.6 mm to (215.6, 118.0), turned to -90 degrees
- moved Q1 190.6 mm to (227.1, 108.1), turned to -90 degrees
- moved L1 178.5 mm to (223.4, 87.5), turned to -90 degrees
- moved D1 173.4 mm to (207.5, 89.2), turned to 0 degrees
- moved Q6 159.5 mm to (214.2, 108.1), turned to -90 degrees
- moved Q4 150.8 mm to (209.9, 108.1), turned to -90 degrees
- moved Q3 147.0 mm to (212.8, 76.2), turned to 90 degrees
- moved U1 142.9 mm to (215.3, 67.9), turned to 180 degrees
- moved R10 142.1 mm to (217.8, 135.1)
- moved R9 141.7 mm to (217.8, 132.1)
- moved R5 140.3 mm to (218.1, 118.1), turned to 90 degrees
- moved Q7 137.6 mm to (216.8, 76.2), turned to 90 degrees
- moved Q8 135.7 mm to (205.8, 108.0), turned to -90 degrees
- moved R4 128.4 mm to (206.3, 72.2)
Connections:
- D1 pad 2: GND -> LiPO Low
- L1 pad 1: Net-(D1-K) -> Net-(D5-K)
- L1 pad 2: Net-(D2-A) -> Switch_Regulated_V
- Q1 pad 1: GND -> LiPO1_Control
- Q1 pad 2: Net-(Q1-B) -> ADC_v-to-c
- Q1 pad 3: Net-(Q1-C) -> Net-(D1-K)
- Q2 pad 1: Net-(D1-K) -> LiPO2_Control
- Q2 pad 2: Net-(Q1-C) -> ADC_v-to-c
- Q2 pad 3: +5V -> LiPO Mid
- Q3 pad 1: Net-(D3-K) -> Switch_Regulator_PWM
- Q3 pad 2: Net-(Q3-G) -> GND
- Q3 pad 3: Net-(D2-A) -> Net-(Q3-D)
- Q4 pad 1: Net-(D3-A) -> LiPO2_Control
- Q4 pad 2: Net-(Q4-G) -> GND
- Q4 pad 3: Net-(D2-A) -> Net-(Q4-D)
- Q6 pad 1: GND -> Net-(Q6-G)
- Q6 pad 2: Net-(Q6-B) -> LiPO Mid
- Q6 pad 3: Net-(Q4-G) -> Switch_Regulated_V
- Q7 pad 1: Net-(Q7-D) -> Net-(Q3-D)
- Q7 pad 2: Net-(Q7-G) -> Net-(D5-K)
- Q7 pad 3: Net-(D3-K) -> USB Vdc
- Q8 pad 1: Net-(Q7-D) -> Net-(Q4-D)
- Q8 pad 2: Net-(Q8-G) -> Net-(D7-A)
- Q8 pad 3: Net-(D4-K) -> Switch_Regulated_V
- R1 pad 1: +5V -> ADC_v-to-c
- R1 pad 2: Net-(Q1-C) -> GND
- R10 pad 2: Net-(U1A--) -> Net-(U3A-INA-)
- R4 pad 1: Net-(Q7-G) -> Net-(U1-EN)
- R4 pad 2: Net-(Q6-B) -> USB Vdc
- R5 pad 1: Net-(Q8-G) -> 3.3v Battery
- R5 pad 2: Net-(Q5-B) -> FB
- R9 pad 1: Net-(U1A--) -> Net-(U3A-INA-)
- R9 pad 2: Net-(H1-Pad1) -> ADC_Current
- U1 pad 1: Net-(H1-Pad1) -> USB Vdc
- U1 pad 2: Net-(U1A--) -> GND
- U1 pad 3: Net-(Q7-D) -> Net-(U1-EN)
- U1 pad 4: (no net) -> unconnected-(U1-NC-Pad4)
- U1 pad 5: (no net) -> MCU Vdd
Routing:
- net GND: track 0.00 -> 315.4 mm, vias 0 -> 14
- net USB Vdc: track 0.00 -> 124.0 mm, vias 0 -> 6
- net MCU Vdd: track 0.00 -> 106.9 mm
- net Switch_Regulated_V: track 0.00 -> 104.7 mm, vias 0 -> 5
- net LiPO1_Control: track 0.00 -> 100.5 mm, vias 0 -> 5
- net Switch_Regulator_PWM: track 0.00 -> 98.2 mm, vias 0 -> 4
- net LiPO2_Control: track 0.00 -> 81.7 mm, vias 0 -> 4
- net LiPO High: track 0.00 -> 78.1 mm, vias 0 -> 4
- net ADC_v-to-c: track 0.00 -> 66.0 mm, vias 0 -> 2
- net LiPO Low: track 0.00 -> 55.5 mm, vias 0 -> 1
- net LiPO Mid: track 0.00 -> 42.8 mm, vias 0 -> 4
- net 3.3v Battery: track 0.00 -> 37.6 mm, vias 0 -> 2
- net ADC_Current: track 0.00 -> 36.2 mm, vias 0 -> 2
- net Net-(D1-K): track 0.00 -> 34.8 mm, vias 0 -> 2
- net Net-(D7-A): track 0.00 -> 28.7 mm, vias 0 -> 2
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Other:
- board outline added: 30 x 100 mm
