File: BatteryCharger/_autosave-462FinalProject.kicad_sch (KiCad schematic)
At the start: 46 parts, among them IC1 TPS562231DRLR, J2 3_Pin_Header_to_Battery, J3 USB_B_Micro, J4 3_Pin_Header_to_IPOD, J5 Conn_01x04_Pin, Q1 MMFTN6001, Q2 MMFTN6001, Q3 SI2302, Q4 SI2302, Q6 BSS84AK,215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

Commit message: "Complete" kicad pcb
Other:
- note added: "pcb board 100mm y 30mm x battery output/input right edge of board"
- note removed: "pcb board 75mm y 35mm x battery output/input right edge of board"
- moved on the sheet: U3B, U3C, U3D
