File: player_system/AUD_OUTPUT_AMP.kicad_sch (KiCad schematic)
At the start: 9 parts, among them Q1 SI2302, Q2 SI2302

Commit message: Nearly done with player PCB
Parts:
- renumbered RN7 to RN5, TP88 to TP86, TP89 to TP87, TP90 to TP88, TP91 to TP89, U4 to U5
Connections:
- net GND: now also RN4.8 (R1.2); no longer RN4.6 (R3.2)
- net at TP86.1, U5.2 (INA-): now also RN4.1 (R1.1), RN4.5 (R4.2); no longer RN4.3 (R3.1), RN4.7 (R2.2)
- net at Q2.3 (D), TP87.1, U5.1 (OUTA): now also RN4.4 (R4.1); no longer RN4.2 (R2.1)
