File: player_system/mic_aud_conditioning_grn.kicad_sch (KiCad schematic)
At the start: 11 parts

Commit message: Nearly done with player PCB
Parts:
- renumbered C3 to C25, R2 to R1, R1 to R2, RN6 to RN3, TP85 to TP83, TP86 to TP84, TP87 to TP85, U2 to U1
Changed lines of the file:
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@@
   (symbol (lib_id "Device:R_Small") (at 68.58 71.12 180) (unit 1)
     (in_bom yes) (on_board yes) (dnp no) (fields_autoplaced)
-    (property "Reference" "R1" (at 71.12 69.85 0)
+    (property "Reference" "R2" (at 71.12 69.85 0)
       (effects (font (size 1.27 1.27)) (justify right))
     )
@@
       (project "player_system"
         (path "/81c17b42-923e-4300-8661-2d9ed419c599/fbc721cf-3662-46b0-aa7e-065032f3a2ab"
-          (reference "R1") (unit 1)
+          (reference "R2") (unit 1)
         )
       )
@@
   (symbol (lib_id "power:+3.3V") (at 62.23 54.61 90) (mirror x) (unit 1)
     (in_bom yes) (on_board yes) (dnp no)
-    (property "Reference" "#PWR041" (at 66.04 54.61 0)
+    (property "Reference" "#PWR086" (at 66.04 54.61 0)
       (effects (font (size 1.27 1.27)) hide)
     )
@@
       (project "player_system"
         (path "/81c17b42-923e-4300-8661-2d9ed419c599/fbc721cf-3662-46b0-aa7e-065032f3a2ab"
-          (reference "#PWR041") (unit 1)
+          (reference "#PWR086") (unit 1)
         )
       )
@@
   (symbol (lib_id "Device:R_Pack04_Split") (at 46.99 55.88 0) (unit 3)
     (in_bom yes) (on_board yes) (dnp no)
-    (property "Reference" "RN6" (at 49.53 58.42 90)
+    (property "Reference" "RN3" (at 49.53 58.42 90)
       (effects (font (size 1.27 1.27)) (justify left))
     )
@@
       (project "player_system"
         (path "/81c17b42-923e-4300-8661-2d9ed419c599/fbc721cf-3662-46b0-aa7e-065032f3a2ab"
-          (reference "RN6") (unit 3)
+          (reference "RN3") (unit 3)
         )
       )
@@
   (symbol (lib_id "power:GND") (at 60.96 73.66 0) (mirror y) (unit 1)
     (in_bom yes) (on_board yes) (dnp no)
-    (property "Reference" "#PWR069" (at 60.96 80.01 0)
+    (property "Reference" "#PWR085" (at 60.96 80.01 0)
       (effects (font (size 1.27 1.27)) hide)
     )
@@
       (project "player_system"
         (path "/81c17b42-923e-4300-8661-2d9ed419c599/fbc721cf-3662-46b0-aa7e-065032f3a2ab"
-          (reference "#PWR069") (unit 1)
+          (reference "#PWR085") (unit 1)
         )
       )
@@
   (symbol (lib_id "RTOS_POD:MCP6489-E/SL") (at 78.74 52.07 0) (mirror x) (unit 1)
     (in_bom yes) (on_board yes) (dnp no)
-    (property "Reference" "U2" (at 86.36 55.88 0)
+    (property "Reference" "U1" (at 86.36 55.88 0)
       (effects (font (size 1.27 1.27)))
     )
@@
       (project "player_system"
         (path "/81c17b42-923e-4300-8661-2d9ed419c599/fbc721cf-3662-46b0-aa7e-065032f3a2ab"
-          (reference "U2") (unit 1)
+          (reference "U1") (unit 1)
         )
       )
@@
   (symbol (lib_id "power:GND") (at 83.82 46.99 0) (mirror x) (unit 1)
     (in_bom yes) (on_board yes) (dnp no)
-    (property "Reference" "#PWR043" (at 83.82 40.64 0)
+    (property "Reference" "#PWR088" (at 83.82 40.64 0)
       (effects (font (size 1.27 1.27)) hide)
     )
@@
       (project "player_system"
         (path "/81c17b42-923e-4300-8661-2d9ed419c599/fbc721cf-3662-46b0-aa7e-065032f3a2ab"
-          (reference "#PWR043") (unit 1)
+          (reference "#PWR088") (unit 1)
         )
       )
@@
   (symbol (lib_id "Connector:TestPoint_Alt") (at 68.58 67.31 0) (unit 1)
     (in_bom yes) (on_board yes) (dnp no)
-    (property "Reference" "TP86" (at 69.088 67.056 90)
+    (property "Reference" "TP84" (at 69.088 67.056 90)
       (effects (font (size 0.5 0.5)) (justify left))
     )
@@
       (project "player_system"
         (path "/81c17b42-923e-4300-8661-2d9ed419c599/fbc721cf-3662-46b0-aa7e-065032f3a2ab"
-          (reference "TP86") (unit 1)
+          (reference "TP84") (unit 1)
         )
       )
@@
   (symbol (lib_id "Connector:TestPoint_Alt") (at 39.37 49.53 180) (unit 1)
     (in_bom yes) (on_board yes) (dnp no)
-    (property "Reference" "TP85" (at 38.862 49.784 90)
+    (property "Reference" "TP83" (at 38.862 49.784 90)
       (effects (font (size 0.5 0.5)) (justify left))
     )
@@
       (project "player_system"
         (path "/81c17b42-923e-4300-8661-2d9ed419c599/fbc721cf-3662-46b0-aa7e-065032f3a2ab"
-          (reference "TP85") (unit 1)
+          (reference "TP83") (unit 1)
         )
       )
@@
   (symbol (lib_id "Device:R_Small") (at 60.96 71.12 180) (unit 1)
     (in_bom yes) (on_board yes) (dnp no) (fields_autoplaced)
-    (property "Reference" "R2" (at 63.5 69.85 0)
+    (property "Reference" "R1" (at 63.5 69.85 0)
       (effects (font (size 1.27 1.27)) (justify right))
     )
@@
       (project "player_system"
         (path "/81c17b42-923e-4300-8661-2d9ed419c599/fbc721cf-3662-46b0-aa7e-065032f3a2ab"
-          (reference "R2") (unit 1)
+          (reference "R1") (unit 1)
         )
       )
@@
   (symbol (lib_id "Device:R_Pack04_Split") (at 36.83 55.88 0) (unit 4)
     (in_bom yes) (on_board yes) (dnp no)
-    (property "Reference" "RN6" (at 34.29 58.42 90)
+    (property "Reference" "RN3" (at 34.29 58.42 90)
       (effects (font (size 1.27 1.27)) (justify left))
     )
@@
       (project "player_system"
         (path "/81c17b42-923e-4300-8661-2d9ed419c599/fbc721cf-3662-46b0-aa7e-065032f3a2ab"
-          (reference "RN6") (unit 4)
+          (reference "RN3") (unit 4)
         )
       )
@@
   (symbol (lib_id "Device:R_Pack04_Split") (at 46.99 43.18 0) (unit 2)
     (in_bom yes) (on_board yes) (dnp no)
-    (property "Reference" "RN6" (at 49.53 45.72 90)
+    (property "Reference" "RN3" (at 49.53 45.72 90)
       (effects (font (size 1.27 1.27)) (justify left))
     )
@@
       (project "player_system"
         (path "/81c17b42-923e-4300-8661-2d9ed419c599/fbc721cf-3662-46b0-aa7e-065032f3a2ab"
-          (reference "RN6") (unit 2)
+          (reference "RN3") (unit 2)
         )
       )
@@
   (symbol (lib_id "Device:R_Pack04_Split") (at 36.83 43.18 0) (mirror y) (unit 1)
     (in_bom yes) (on_board yes) (dnp no)
-    (property "Reference" "RN6" (at 34.29 45.72 90)
+    (property "Reference" "RN3" (at 34.29 45.72 90)
       (effects (font (size 1.27 1.27)) (justify left))
     )
@@
       (project "player_system"
         (path "/81c17b42-923e-4300-8661-2d9ed419c599/fbc721cf-3662-46b0-aa7e-065032f3a2ab"
-          (reference "RN6") (unit 1)
+          (reference "RN3") (unit 1)
         )
       )
@@
   (symbol (lib_id "power:GND") (at 68.58 73.66 0) (mirror y) (unit 1)
     (in_bom yes) (on_board yes) (dnp no)
-    (property "Reference" "#PWR042" (at 68.58 80.01 0)
+    (property "Reference" "#PWR087" (at 68.58 80.01 0)
       (effects (font (size 1.27 1.27)) hide)
     )
@@
       (project "player_system"
         (path "/81c17b42-923e-4300-8661-2d9ed419c599/fbc721cf-3662-46b0-aa7e-065032f3a2ab"
-          (reference "#PWR042") (unit 1)
+          (reference "#PWR087") (unit 1)
         )
       )
@@
   (symbol (lib_id "Device:C_Small") (at 41.91 49.53 90) (unit 1)
     (in_bom yes) (on_board yes) (dnp no) (fields_autoplaced)
-    (property "Reference" "C3" (at 41.9163 43.18 90)
+    (property "Reference" "C25" (at 41.9163 43.18 90)
       (effects (font (size 1.27 1.27)))
     )
@@
       (project "player_system"
         (path "/81c17b42-923e-4300-8661-2d9ed419c599/fbc721cf-3662-46b0-aa7e-065032f3a2ab"
-          (reference "C3") (unit 1)
+          (reference "C25") (unit 1)
         )
       )
@@
   (symbol (lib_id "Connector:TestPoint_Alt") (at 76.2 49.53 0) (unit 1)
     (in_bom yes) (on_board yes) (dnp no)
-    (property "Reference" "TP87" (at 76.708 49.276 90)
+    (property "Reference" "TP85" (at 76.708 49.276 90)
       (effects (font (size 0.5 0.5)) (justify left))
     )
@@
       (project "player_system"
         (path "/81c17b42-923e-4300-8661-2d9ed419c599/fbc721cf-3662-46b0-aa7e-065032f3a2ab"
-          (reference "TP87") (unit 1)
+          (reference "TP85") (unit 1)
         )
       )
@@
   (symbol (lib_id "power:GND") (at 46.99 63.5 0) (mirror y) (unit 1)
     (in_bom yes) (on_board yes) (dnp no)
-    (property "Reference" "#PWR040" (at 46.99 69.85 0)
+    (property "Reference" "#PWR084" (at 46.99 69.85 0)
       (effects (font (size 1.27 1.27)) hide)
     )
@@
       (project "player_system"
         (path "/81c17b42-923e-4300-8661-2d9ed419c599/fbc721cf-3662-46b0-aa7e-065032f3a2ab"
-          (reference "#PWR040") (unit 1)
+          (reference "#PWR084") (unit 1)
         )
       )
@@
   (symbol (lib_id "power:+3.3V") (at 83.82 57.15 0) (mirror x) (unit 1)
     (in_bom yes) (on_board yes) (dnp no)
-    (property "Reference" "#PWR044" (at 83.82 53.34 0)
+    (property "Reference" "#PWR089" (at 83.82 53.34 0)
       (effects (font (size 1.27 1.27)) hide)
     )
@@
       (project "player_system"
         (path "/81c17b42-923e-4300-8661-2d9ed419c599/fbc721cf-3662-46b0-aa7e-065032f3a2ab"
-          (reference "#PWR044") (unit 1)
+          (reference "#PWR089") (unit 1)
         )
       )
@@
   (symbol (lib_id "power:+3.3V") (at 46.99 35.56 0) (mirror y) (unit 1)
     (in_bom yes) (on_board yes) (dnp no)
-    (property "Reference" "#PWR039" (at 46.99 39.37 0)
+    (property "Reference" "#PWR083" (at 46.99 39.37 0)
       (effects (font (size 1.27 1.27)) hide)
     )
@@
       (project "player_system"
         (path "/81c17b42-923e-4300-8661-2d9ed419c599/fbc721cf-3662-46b0-aa7e-065032f3a2ab"
-          (reference "#PWR039") (unit 1)
-        )
-      )
+          (reference "#PWR083") (unit 1)
+        )
+      )
