File: player_system/player_system.kicad_sch (KiCad schematic)
At the start: 122 parts, among them U1 STM32G474VEHx, U3 STM32G030F6Px, Y1 16mhz

Commit message: Nearly done with player PCB
Parts:
- removed NT1: NetTie_2, NetTie:NetTie-2_SMD_Pad0.5mm, symbol Device:NetTie_2
- removed RN3, RN4, RN5: 10k, Resistor_SMD:R_Array_Concave_4x0603, symbol Device:R_Pack04_Split
- added C10, C11, C12, C13, C14, C15, C16, C17, C18, C19, C20, C21, C22, C23, C24, C7, C8, C9: 10uf, Capacitor_SMD:C_0805_2012Metric_Pad1.18x1.45mm_HandSolder, symbol Device:C_Small
- added C4, C6: 100n, Capacitor_SMD:C_0805_2012Metric_Pad1.18x1.45mm_HandSolder, symbol Device:C_Small
- added H1, H10, H11, H12, H2, H3, H4, H5, H6, H7, H8, H9: MountingHole, MountingHole:MountingHole_2.2mm_M2, symbol Mechanical:MountingHole
- added SW2, SW4: ~, Button_Switch_SMD:SW_SPST_EVPBF, symbol Switch:SW_Push
- added U4: LDI1117-05H, Package_TO_SOT_SMD:SOT-223-3_TabPin2, symbol Regulator_Linear:AP1117-15
- C1, C2: value C_Small -> 10pf C0G 2%
- SD_DAT1, SD_DAT2: footprint TestPoint:TestPoint_Loop_D2.50mm_Drill1.85mm -> rtospod_footprints:tht_testpt
- Y1: value 16mhz -> 16mhz 10ppm; footprint (none) -> Crystal:Crystal_SMD_2520-4Pin_2.5x2.0mm
- renumbered AUD_GND2 to AUD_GND1, AUD_GND1 to AUD_GND2, AUD_GND4 to AUD_GND3, AUD_GND3 to AUD_GND4, C4 to C3, SW2 to SW3, TP3 to TP1, TP12 to TP10, TP13 to TP11, TP14 to TP12, TP15 to TP13, TP16 to TP14, TP17 to TP15, TP18 to TP16, TP19 to TP17, TP20 to TP18, TP21 to TP19, TP4 to TP2, TP22 to TP20, TP23 to TP21, TP24 to TP22, TP25 to TP23, TP26 to TP24, TP27 to TP25, TP28 to TP26, TP29 to TP27, TP30 to TP28, TP31 to TP29, TP5 to TP3, TP32 to TP30, TP33 to TP31, TP34 to TP32, TP35 to TP33, TP36 to TP34, TP37 to TP35, TP38 to TP36, TP39 to TP37, TP40 to TP38, TP41 to TP39, TP6 to TP4, TP42 to TP40, TP43 to TP41, TP44 to TP42, TP45 to TP43, TP46 to TP44, TP47 to TP45, TP48 to TP46, TP49 to TP47, TP50 to TP48, TP51 to TP49, TP7 to TP5, TP52 to TP50, TP53 to TP51, TP54 to TP52, TP55 to TP53, TP56 to TP54, TP57 to TP55, TP58 to TP56, TP59 to TP57, TP60 to TP58, TP61 to TP59, TP8 to TP6, TP62 to TP60, TP63 to TP61, TP64 to TP62, TP65 to TP63, TP66 to TP64, TP67 to TP65, TP68 to TP66, TP69 to TP67, TP70 to TP68, TP71 to TP69, TP9 to TP7, TP72 to TP70, TP73 to TP71, TP74 to TP72, TP75 to TP73, TP76 to TP74, TP77 to TP75, TP78 to TP76, TP79 to TP77, TP80 to TP78, TP81 to TP79, TP10 to TP8, TP82 to TP80, TP83 to TP81, TP84 to TP82, TP11 to TP9, U2 to U1, U1 to U2
Connections:
- net +3.3V: now also C11.1, C12.1, C13.1, C15.1, C16.1, C17.1, C19.1, C20.1, C21.1, C22.1, C23.1, C24.1, C7.1, C8.1, C9.1
- net +BATT: now also C10.1, U4.3 (VI)
- net GND: now also C10.2, C11.2, C12.2, C13.2, C14.2, C15.2, C16.2, C17.2, C18.2, C19.2, C20.2, C21.2, C22.2, C23.2, C24.2, C4.2, C6.2, C7.2, C8.2, C9.2, SW2.2, SW4.2, U4.1 (GND)
- net PA10: now also C5.1, SW3.1
- net PA11: now also C4.1, SW2.1
- net PA12: now also C6.1, SW4.1
- net PA8: now also C3.1, SW1.1
- net QUADSPI_CLK: now also U2.E4 (PF10); no longer U2.K6 (PE10)
- net at C1.2, U2.E1 (PF0), Y1.2: now also Y1.3 (2)
- net at C2.1, U2.E2 (PF1), Y1.1: now also Y1.4 (1)
- net PF10 renamed PE10
- net PE10: now also U2.K6 (PE10); no longer U2.E4 (PF10)
- new net +5V: C14.1, C18.1, U4.2 (VO)
- no-connect marks 10 -> 2
Other:
- note added: "ADD bridge NRST pin"
- note added: "Filter Caps"
- note added: "Pushbuttons"
- moved on the sheet: AUD_BLACK1, AUD_GND1, AUD_GND2, AUD_GND3, AUD_GND4, AUD_GREEN1, AUD_ORANGE1, AUD_PINK1, C3, C5, GNDDET1, J1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

Commit message: Getting DAC DMA set up
Other:
- note removed: "ADD bridge NRST pin"
Changed lines of the file:
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@@
     (effects (font (size 1.27 1.27) (color 0 0 0 1)) (justify left top))
   )
-  (text_box "* Preamp Audio is boosted by factor of 2\n* Max output voltage is 5v, so preamp audio output should not exceed 2.5v.\n* Trimmable gain from 1 to 40\n* If this is not an appropriate range, we can consider Changing the resistors\n* Will need to be carefully trimmed in bost bias and gain to get good output"
+  (text_box "* Preamp Audio is boosted by factor of 2\n* Max output voltage is 5v, so preamp audio output should not exceed 2.5v.\n* Trimmable gain from 1 to 40\n* If this is not an appropriate range, we can consider Changing the resistors\n* Will need to be carefully trimmed in both bias and gain to get good output"
     (at 252.73 226.06 0) (size 54.61 35.56)
     (stroke (width 0) (type default))
@@
     (effects (font (size 3 3) (thickness 0.6) bold) (justify left bottom))
   )
-  (text "ADD bridge NRST pin" (at 64.77 364.49 0)
-    (effects (font (size 1.27 1.27)) (justify left bottom))
-  )
   (text "Volume Wheel" (at 322.58 41.91 0)

Commit message: Fix PCB Mistake: Crystal Oscilator has two GND pins, not shared pins
Connections:
- net GND: now also Y1.2, Y1.4 (1)
- net at C1.2, U2.E1 (PF0), Y1.3 (2): no longer Y1.2
- net at C2.1, U2.E2 (PF1), Y1.1: no longer Y1.4 (1)
Changed lines of the file:
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@@
     )
   )
+  (symbol (lib_id "power:GND") (at 22.86 40.64 270) (unit 1)
+    (in_bom yes) (on_board yes) (dnp no)
+    (property "Reference" "#PWR037" (at 16.51 40.64 0)
+      (effects (font (size 1.27 1.27)) hide)
+    )
+    (property "Value" "GND" (at 22.86 43.18 0)
+      (effects (font (size 1.27 1.27)) hide)
+    )
+    (property "Footprint" "" (at 22.86 40.64 0)
+      (effects (font (size 1.27 1.27)) hide)
+    )
+    (property "Datasheet" "" (at 22.86 40.64 0)
+      (effects (font (size 1.27 1.27)) hide)
+    )
+    (pin "1")
+    (instances
+      (project "player_system"
+        (path "/81c17b42-923e-4300-8661-2d9ed419c599"
+          (reference "#PWR037") (unit 1)
+        )
+      )
+    )
+  )
   (symbol (lib_id "power:+3.3V") (at 313.69 102.87 0) (unit 1)
     (in_bom yes) (on_board yes) (dnp no)
@@
   (symbol (lib_id "Device:Crystal_Small") (at 26.67 40.64 270) (mirror x) (unit 1)
     (in_bom yes) (on_board yes) (dnp no)
-    (property "Reference" "Y1" (at 20.32 40.64 90)
+    (property "Reference" "Y1" (at 29.21 41.91 0)
       (effects (font (size 1.27 1.27)) (justify left))
     )
-    (property "Value" "16mhz 10ppm" (at 17.78 38.1 90)
+    (property "Value" "16mhz 10ppm" (at 12.7 38.1 90)
       (effects (font (size 1.27 1.27)) (justify left))
     )
